File: Eurocard_3U_VME/Eurocard_3U_VME.sch (KiCad schematic (older format))
At the start: 1 part, among them J1 VG64_VME_3Rows_3x32_J1_P1

Commit message: Update 3U from 6U
Parts:
- added J2: VG64_VME_3Rows_3x32_J2_P2, d_connectors:DIN41612_B_3x32_Horizontal, symbol d_connectors:VG64_VME_3Rows_3x32_J1_P1
Changed lines of the file:
@@
 $EndDescr
+$Comp
+L d_connectors:VG64_VME_3Rows_3x32_J1_P1 J1
+U 1 1 5DDFD772
+P 1200 2500
+F 0 "J1" H 1280 2492 50  0000 L CNN
+F 1 "VG64_VME_3Rows_3x32_J1_P1" H 1280 2401 50  0000 L CNN
+F 2 "d_connectors:DIN41612_B_3x32_Horizontal" H 1200 2500 50  0001 C CNN
+F 3 "~" H 1200 2500 50  0001 C CNN
+	1    1200 2500
+	1    0    0    -1
+$EndComp
+$Comp
+L d_connectors:VG64_VME_3Rows_3x32_J1_P1 J1
+U 2 1 5DE12553
+P 2700 2500
+F 0 "J1" H 2780 2492 50  0000 L CNN
+F 1 "VG64_VME_3Rows_3x32_J1_P1" H 2780 2401 50  0000 L CNN
+F 2 "d_connectors:DIN41612_B_3x32_Horizontal" H 2700 2500 50  0001 C CNN
+F 3 "~" H 2700 2500 50  0001 C CNN
+	2    2700 2500
+	1    0    0    -1
+$EndComp
+$Comp
+L d_connectors:VG64_VME_3Rows_3x32_J1_P1 J1
+U 3 1 5DE1ECAF
+P 4200 2500
+F 0 "J1" H 4280 2492 50  0000 L CNN
+F 1 "VG64_VME_3Rows_3x32_J1_P1" H 4280 2401 50  0000 L CNN
+F 2 "d_connectors:DIN41612_B_3x32_Horizontal" H 4200 2500 50  0001 C CNN
+F 3 "~" H 4200 2500 50  0001 C CNN
+	3    4200 2500
+	1    0    0    -1
+$EndComp
+$Comp
+L d_connectors:VG64_VME_3Rows_3x32_J1_P1 J2
+U 1 1 5DE28E89
+P 6700 2500
+F 0 "J2" H 6780 2492 50  0000 L CNN
+F 1 "VG64_VME_3Rows_3x32_J2_P2" H 6780 2401 50  0000 L CNN
+F 2 "d_connectors:DIN41612_B_3x32_Horizontal" H 6700 2500 50  0001 C CNN
+F 3 "~" H 6700 2500 50  0001 C CNN
+	1    6700 2500
+	1    0    0    -1
+$EndComp
+$Comp
+L d_connectors:VG64_VME_3Rows_3x32_J1_P1 J2
+U 2 1 5DE30083
+P 8200 2500
+F 0 "J2" H 8280 2492 50  0000 L CNN
+F 1 "VG64_VME_3Rows_3x32_J2_P2" H 8280 2401 50  0000 L CNN
+F 2 "d_connectors:DIN41612_B_3x32_Horizontal" H 8200 2500 50  0001 C CNN
+F 3 "~" H 8200 2500 50  0001 C CNN
+	2    8200 2500
+	1    0    0    -1
+$EndComp
+$Comp
+L d_connectors:VG64_VME_3Rows_3x32_J1_P1 J2
+U 3 1 5DE3759B
+P 9700 2500
+F 0 "J2" H 9780 2492 50  0000 L CNN
+F 1 "VG64_VME_3Rows_3x32_J2_P2" H 9780 2401 50  0000 L CNN
+F 2 "d_connectors:DIN41612_B_3x32_Horizontal" H 9700 2500 50  0001 C CNN
+F 3 "~" H 9700 2500 50  0001 C CNN
+	3    9700 2500
+	1    0    0    -1
+$EndComp
+$Comp
+L power:GND #PWR?
+U 1 1 5DDF0127
+P 1000 1800
+F 0 "#PWR?" H 1000 1550 50  0001 C CNN
+F 1 "GND" V 1005 1672 50  0000 R CNN
+F 2 "" H 1000 1800 50  0001 C CNN
+F 3 "" H 1000 1800 50  0001 C CNN
+	1    1000 1800
+	0    1    1    0
+$EndComp
+$Comp
+L power:GND #PWR?
+U 1 1 5DDF0B5B
+P 4000 1800
+F 0 "#PWR?" H 4000 1550 50  0001 C CNN
+F 1 "GND" V 4005 1672 50  0000 R CNN
+F 2 "" H 4000 1800 50  0001 C CNN
+F 3 "" H 4000 1800 50  0001 C CNN
+	1    4000 1800
+	0    1    1    0
+$EndComp
+$Comp
+L power:GND #PWR?
+U 1 1 5DDF167D
+P 1000 2000
+F 0 "#PWR?" H 1000 1750 50  0001 C CNN
+F 1 "GND" V 1005 1872 50  0000 R CNN
+F 2 "" H 1000 2000 50  0001 C CNN
+F 3 "" H 1000 2000 50  0001 C CNN
+	1    1000 2000
+	0    1    1    0
+$EndComp
+$Comp
+L power:GND #PWR?
+U 1 1 5DDF2337
+P 1000 2400
+F 0 "#PWR?" H 1000 2150 50  0001 C CNN
+F 1 "GND" V 1005 2272 50  0000 R CNN
+F 2 "" H 1000 2400 50  0001 C CNN
+F 3 "" H 1000 2400 50  0001 C CNN
+	1    1000 2400
+	0    1    1    0
+$EndComp
+$Comp
+L power:GND #PWR?
+U 1 1 5DDF2E48
+P 1000 2600
+F 0 "#PWR?" H 1000 2350 50  0001 C CNN
+F 1 "GND" V 1005 2472 50  0000 R CNN
+F 2 "" H 1000 2600 50  0001 C CNN
+F 3 "" H 1000 2600 50  0001 C CNN
+	1    1000 2600
+	0    1    1    0
+$EndComp
+$Comp
+L power:GND #PWR?
+U 1 1 5DDF34B3
+P 1000 2800
+F 0 "#PWR?" H 1000 2550 50  0001 C CNN
+F 1 "GND" V 1005 2672 50  0000 R CNN
+F 2 "" H 1000 2800 50  0001 C CNN
+F 3 "" H 1000 2800 50  0001 C CNN
+	1    1000 2800
+	0    1    1    0
+$EndComp
+$Comp
+L power:GND #PWR?
+U 1 1 5DDF3A63
+P 2500 2900
+F 0 "#PWR?" H 2500 2650 50  0001 C CNN
+F 1 "GND" V 2505 2772 50  0000 R CNN
+F 2 "" H 2500 2900 50  0001 C CNN
+F 3 "" H 2500 2900 50  0001 C CNN
+	1    2500 2900
+	0    1    1    0
+$EndComp
+$Comp
+L power:GND #PWR?
+U 1 1 5DDF47FA
+P 2500 3200
+F 0 "#PWR?" H 2500 2950 50  0001 C CNN
+F 1 "GND" V 2505 3072 50  0000 R CNN
+F 2 "" H 2500 3200 50  0001 C CNN
+F 3 "" H 2500 3200 50  0001 C CNN
+	1    2500 3200
+	0    1    1    0
+$EndComp
+$Comp
+L power:+5V #PWR?
+U 1 1 5DDF5905
+P 1000 4100
+F 0 "#PWR?" H 1000 3950 50  0001 C CNN
+F 1 "+5V" V 1015 4228 50  0000 L CNN
+F 2 "" H 1000 4100 50  0001 C CNN
+F 3 "" H 1000 4100 50  0001 C CNN
+	1    1000 4100
+	0    -1   -1   0
+$EndComp
+$Comp
+L power:+5V #PWR?
+U 1 1 5DDF6272
+P 2500 4100
+F 0 "#PWR?" H 2500 3950 50  0001 C CNN
+F 1 "+5V" V 2515 4228 50  0000 L CNN
+F 2 "" H 2500 4100 50  0001 C CNN
+F 3 "" H 2500 4100 50  0001 C CNN
+	1    2500 4100
+	0    -1   -1   0
+$EndComp
+$Comp
+L power:+5V #PWR?
+U 1 1 5DDF69EC
+P 4000 4100
+F 0 "#PWR?" H 4000 3950 50  0001 C CNN
+F 1 "+5V" V 4015 4228 50  0000 L CNN
+F 2 "" H 4000 4100 50  0001 C CNN
+F 3 "" H 4000 4100 50  0001 C CNN
+	1    4000 4100
+	0    -1   -1   0
+$EndComp
+$Comp
+L power:+12V #PWR?
+U 1 1 5DDF80AE
+P 4000 4000
+F 0 "#PWR?" H 4000 3850 50  0001 C CNN
+F 1 "+12V" V 4015 4128 50  0000 L CNN
+F 2 "" H 4000 4000 50  0001 C CNN
+F 3 "" H 4000 4000 50  0001 C CNN
+	1    4000 4000
+	0    -1   -1   0
+$EndComp
 $Comp
 L power:-12V #PWR?
@@
 	0    -1   -1   0
 $EndComp
-$Comp
-L power:+12V #PWR?
-U 1 1 5DDF80AE
-P 4000 4000
-F 0 "#PWR?" H 4000 3850 50  0001 C CNN
-F 1 "+12V" V 4015 4128 50  0000 L CNN
-F 2 "" H 4000 4000 50  0001 C CNN
-F 3 "" H 4000 4000 50  0001 C CNN
-	1    4000 4000
-	0    -1   -1   0
-$EndComp
-$Comp
-L power:+5V #PWR?
-U 1 1 5DDF69EC
-P 4000 4100
-F 0 "#PWR?" H 4000 3950 50  0001 C CNN
-F 1 "+5V" V 4015 4228 50  0000 L CNN
-F 2 "" H 4000 4100 50  0001 C CNN
-F 3 "" H 4000 4100 50  0001 C CNN
-	1    4000 4100
-	0    -1   -1   0
-$EndComp
-$Comp
-L power:+5V #PWR?
-U 1 1 5DDF6272
-P 2500 4100
-F 0 "#PWR?" H 2500 3950 50  0001 C CNN
-F 1 "+5V" V 2515 4228 50  0000 L CNN
-F 2 "" H 2500 4100 50  0001 C CNN
-F 3 "" H 2500 4100 50  0001 C CNN
-	1    2500 4100
-	0    -1   -1   0
-$EndComp
-$Comp
-L power:+5V #PWR?
-U 1 1 5DDF5905
-P 1000 4100
-F 0 "#PWR?" H 1000 3950 50  0001 C CNN
-F 1 "+5V" V 1015 4228 50  0000 L CNN
-F 2 "" H 1000 4100 50  0001 C CNN
-F 3 "" H 1000 4100 50  0001 C CNN
-	1    1000 4100
-	0    -1   -1   0
-$EndComp
-$Comp
-L power:GND #PWR?
-U 1 1 5DDF47FA
-P 2500 3200
-F 0 "#PWR?" H 2500 2950 50  0001 C CNN
-F 1 "GND" V 2505 3072 50  0000 R CNN
-F 2 "" H 2500 3200 50  0001 C CNN
-F 3 "" H 2500 3200 50  0001 C CNN
-	1    2500 3200
-	0    1    1    0
-$EndComp
-$Comp
-L power:GND #PWR?
-U 1 1 5DDF3A63
-P 2500 2900
-F 0 "#PWR?" H 2500 2650 50  0001 C CNN
-F 1 "GND" V 2505 2772 50  0000 R CNN
-F 2 "" H 2500 2900 50  0001 C CNN
-F 3 "" H 2500 2900 50  0001 C CNN
-	1    2500 2900
-	0    1    1    0
-$EndComp
-$Comp
-L power:GND #PWR?
-U 1 1 5DDF34B3
-P 1000 2800
-F 0 "#PWR?" H 1000 2550 50  0001 C CNN
-F 1 "GND" V 1005 2672 50  0000 R CNN
-F 2 "" H 1000 2800 50  0001 C CNN
-F 3 "" H 1000 2800 50  0001 C CNN
-	1    1000 2800
-	0    1    1    0
-$EndComp
-$Comp
-L power:GND #PWR?
-U 1 1 5DDF2E48
-P 1000 2600
-F 0 "#PWR?" H 1000 2350 50  0001 C CNN
-F 1 "GND" V 1005 2472 50  0000 R CNN
-F 2 "" H 1000 2600 50  0001 C CNN
-F 3 "" H 1000 2600 50  0001 C CNN
-	1    1000 2600
-	0    1    1    0
-$EndComp
-$Comp
-L power:GND #PWR?
-U 1 1 5DDF2337
-P 1000 2400
-F 0 "#PWR?" H 1000 2150 50  0001 C CNN
-F 1 "GND" V 1005 2272 50  0000 R CNN
-F 2 "" H 1000 2400 50  0001 C CNN
-F 3 "" H 1000 2400 50  0001 C CNN
-	1    1000 2400
-	0    1    1    0
-$EndComp
-$Comp
-L power:GND #PWR?
-U 1 1 5DDF167D
-P 1000 2000
-F 0 "#PWR?" H 1000 1750 50  0001 C CNN
-F 1 "GND" V 1005 1872 50  0000 R CNN
-F 2 "" H 1000 2000 50  0001 C CNN
-F 3 "" H 1000 2000 50  0001 C CNN
-	1    1000 2000
-	0    1    1    0
-$EndComp
-$Comp
-L power:GND #PWR?
-U 1 1 5DDF0B5B
-P 4000 1800
-F 0 "#PWR?" H 4000 1550 50  0001 C CNN
-F 1 "GND" V 4005 1672 50  0000 R CNN
-F 2 "" H 4000 1800 50  0001 C CNN
-F 3 "" H 4000 1800 50  0001 C CNN
-	1    4000 1800
-	0    1    1    0
-$EndComp
-$Comp
-L power:GND #PWR?
-U 1 1 5DDF0127
-P 1000 1800
-F 0 "#PWR?" H 1000 1550 50  0001 C CNN
-F 1 "GND" V 1005 1672 50  0000 R CNN
-F 2 "" H 1000 1800 50  0001 C CNN
-F 3 "" H 1000 1800 50  0001 C CNN
-	1    1000 1800
-	0    1    1    0
-$EndComp
-$Comp
-L d_connectors:VG64_VME_3Rows_3x32_J1_P1 J1
-U 3 1 5DE1ECAF
-P 4200 2500
-F 0 "J1" H 4280 2492 50  0000 L CNN
-F 1 "VG64_VME_3Rows_3x32_J1_P1" H 4280 2401 50  0000 L CNN
-F 2 "d_connectors:DIN41612_B_3x32_Horizontal" H 4200 2500 50  0001 C CNN
-F 3 "~" H 4200 2500 50  0001 C CNN
-	3    4200 2500
-	1    0    0    -1
-$EndComp
-$Comp
-L d_connectors:VG64_VME_3Rows_3x32_J1_P1 J1
-U 2 1 5DE12553
-P 2700 2500
-F 0 "J1" H 2780 2492 50  0000 L CNN
-F 1 "VG64_VME_3Rows_3x32_J1_P1" H 2780 2401 50  0000 L CNN
-F 2 "d_connectors:DIN41612_B_3x32_Horizontal" H 2700 2500 50  0001 C CNN
-F 3 "~" H 2700 2500 50  0001 C CNN
-	2    2700 2500
-	1    0    0    -1
-$EndComp
-$Comp
-L d_connectors:VG64_VME_3Rows_3x32_J1_P1 J1
-U 1 1 5DDFD772
-P 1200 2500
-F 0 "J1" H 1280 2492 50  0000 L CNN
-F 1 "VG64_VME_3Rows_3x32_J1_P1" H 1280 2401 50  0000 L CNN
-F 2 "d_connectors:DIN41612_B_3x32_Horizontal" H 1200 2500 50  0001 C CNN
-F 3 "~" H 1200 2500 50  0001 C CNN
-	1    1200 2500
-	1    0    0    -1
-$EndComp
 $EndSCHEMATC

Commit message: Cut the card and change some dimmensions to adapt to single height VME boards
Parts:
- removed J2: VG64_VME_3Rows_3x32_J2_P2, d_connectors:DIN41612_B_3x32_Horizontal, symbol d_connectors:VG64_VME_3Rows_3x32_J1_P1
Connections:
- net labels removed: +12V, +5V, -12V, GND
Changed lines of the file:
@@
 	1    0    0    -1
 $EndComp
-$Comp
-L d_connectors:VG64_VME_3Rows_3x32_J1_P1 J2
-U 1 1 5DE28E89
-P 6700 2500
-F 0 "J2" H 6780 2492 50  0000 L CNN
-F 1 "VG64_VME_3Rows_3x32_J2_P2" H 6780 2401 50  0000 L CNN
-F 2 "d_connectors:DIN41612_B_3x32_Horizontal" H 6700 2500 50  0001 C CNN
-F 3 "~" H 6700 2500 50  0001 C CNN
-	1    6700 2500
-	1    0    0    -1
-$EndComp
-$Comp
-L d_connectors:VG64_VME_3Rows_3x32_J1_P1 J2
-U 2 1 5DE30083
-P 8200 2500
-F 0 "J2" H 8280 2492 50  0000 L CNN
-F 1 "VG64_VME_3Rows_3x32_J2_P2" H 8280 2401 50  0000 L CNN
-F 2 "d_connectors:DIN41612_B_3x32_Horizontal" H 8200 2500 50  0001 C CNN
-F 3 "~" H 8200 2500 50  0001 C CNN
-	2    8200 2500
-	1    0    0    -1
-$EndComp
-$Comp
-L d_connectors:VG64_VME_3Rows_3x32_J1_P1 J2
-U 3 1 5DE3759B
-P 9700 2500
-F 0 "J2" H 9780 2492 50  0000 L CNN
-F 1 "VG64_VME_3Rows_3x32_J2_P2" H 9780 2401 50  0000 L CNN
-F 2 "d_connectors:DIN41612_B_3x32_Horizontal" H 9700 2500 50  0001 C CNN
-F 3 "~" H 9700 2500 50  0001 C CNN
-	3    9700 2500
-	1    0    0    -1
-$EndComp
-$Comp
-L power:GND #PWR?
-U 1 1 5DDF0127
-P 1000 1800
-F 0 "#PWR?" H 1000 1550 50  0001 C CNN
-F 1 "GND" V 1005 1672 50  0000 R CNN
-F 2 "" H 1000 1800 50  0001 C CNN
-F 3 "" H 1000 1800 50  0001 C CNN
-	1    1000 1800
-	0    1    1    0
-$EndComp
-$Comp
-L power:GND #PWR?
-U 1 1 5DDF0B5B
-P 4000 1800
-F 0 "#PWR?" H 4000 1550 50  0001 C CNN
-F 1 "GND" V 4005 1672 50  0000 R CNN
-F 2 "" H 4000 1800 50  0001 C CNN
-F 3 "" H 4000 1800 50  0001 C CNN
-	1    4000 1800
-	0    1    1    0
-$EndComp
-$Comp
-L power:GND #PWR?
-U 1 1 5DDF167D
-P 1000 2000
-F 0 "#PWR?" H 1000 1750 50  0001 C CNN
-F 1 "GND" V 1005 1872 50  0000 R CNN
-F 2 "" H 1000 2000 50  0001 C CNN
-F 3 "" H 1000 2000 50  0001 C CNN
-	1    1000 2000
-	0    1    1    0
-$EndComp
-$Comp
-L power:GND #PWR?
-U 1 1 5DDF2337
-P 1000 2400
-F 0 "#PWR?" H 1000 2150 50  0001 C CNN
-F 1 "GND" V 1005 2272 50  0000 R CNN
-F 2 "" H 1000 2400 50  0001 C CNN
-F 3 "" H 1000 2400 50  0001 C CNN
-	1    1000 2400
-	0    1    1    0
-$EndComp
-$Comp
-L power:GND #PWR?
-U 1 1 5DDF2E48
-P 1000 2600
-F 0 "#PWR?" H 1000 2350 50  0001 C CNN
-F 1 "GND" V 1005 2472 50  0000 R CNN
-F 2 "" H 1000 2600 50  0001 C CNN
-F 3 "" H 1000 2600 50  0001 C CNN
-	1    1000 2600
-	0    1    1    0
-$EndComp
-$Comp
-L power:GND #PWR?
-U 1 1 5DDF34B3
-P 1000 2800
-F 0 "#PWR?" H 1000 2550 50  0001 C CNN
-F 1 "GND" V 1005 2672 50  0000 R CNN
-F 2 "" H 1000 2800 50  0001 C CNN
-F 3 "" H 1000 2800 50  0001 C CNN
-	1    1000 2800
-	0    1    1    0
-$EndComp
-$Comp
-L power:GND #PWR?
-U 1 1 5DDF3A63
-P 2500 2900
-F 0 "#PWR?" H 2500 2650 50  0001 C CNN
-F 1 "GND" V 2505 2772 50  0000 R CNN
-F 2 "" H 2500 2900 50  0001 C CNN
-F 3 "" H 2500 2900 50  0001 C CNN
-	1    2500 2900
-	0    1    1    0
-$EndComp
-$Comp
-L power:GND #PWR?
-U 1 1 5DDF47FA
-P 2500 3200
-F 0 "#PWR?" H 2500 2950 50  0001 C CNN
-F 1 "GND" V 2505 3072 50  0000 R CNN
-F 2 "" H 2500 3200 50  0001 C CNN
-F 3 "" H 2500 3200 50  0001 C CNN
-	1    2500 3200
-	0    1    1    0
-$EndComp
-$Comp
-L power:+5V #PWR?
-U 1 1 5DDF5905
-P 1000 4100
-F 0 "#PWR?" H 1000 3950 50  0001 C CNN
-F 1 "+5V" V 1015 4228 50  0000 L CNN
-F 2 "" H 1000 4100 50  0001 C CNN
-F 3 "" H 1000 4100 50  0001 C CNN
-	1    1000 4100
-	0    -1   -1   0
-$EndComp
-$Comp
-L power:+5V #PWR?
-U 1 1 5DDF6272
-P 2500 4100
-F 0 "#PWR?" H 2500 3950 50  0001 C CNN
-F 1 "+5V" V 2515 4228 50  0000 L CNN
-F 2 "" H 2500 4100 50  0001 C CNN
-F 3 "" H 2500 4100 50  0001 C CNN
-	1    2500 4100
-	0    -1   -1   0
-$EndComp
-$Comp
-L power:+5V #PWR?
-U 1 1 5DDF69EC
-P 4000 4100
-F 0 "#PWR?" H 4000 3950 50  0001 C CNN
-F 1 "+5V" V 4015 4228 50  0000 L CNN
-F 2 "" H 4000 4100 50  0001 C CNN
-F 3 "" H 4000 4100 50  0001 C CNN
-	1    4000 4100
-	0    -1   -1   0
-$EndComp
-$Comp
-L power:+12V #PWR?
-U 1 1 5DDF80AE
-P 4000 4000
-F 0 "#PWR?" H 4000 3850 50  0001 C CNN
-F 1 "+12V" V 4015 4128 50  0000 L CNN
-F 2 "" H 4000 4000 50  0001 C CNN
-F 3 "" H 4000 4000 50  0001 C CNN
-	1    4000 4000
-	0    -1   -1   0
-$EndComp
-$Comp
-L power:-12V #PWR?
-U 1 1 5DDF9E4E
-P 1000 4000
-F 0 "#PWR?" H 1000 4100 50  0001 C CNN
-F 1 "-12V" V 1015 4128 50  0000 L CNN
-F 2 "" H 1000 4000 50  0001 C CNN
-F 3 "" H 1000 4000 50  0001 C CNN
-	1    1000 4000
-	0    -1   -1   0
-$EndComp
 $EndSCHEMATC
